File: pcb/watertemp_v1.sch (KiCad schematic (older format))
At the start: 14 parts, among them J1 CONN_02X10, U1 LPC11U24FBD48, U2 LP5907-Q1, U3 RN2483, U4 SHT21, U5 DS18B20, Y1 Crystal

Commit message: Add LEDs
Parts:
- added D1, D2, D3: LED, symbol LED_Small
- added R2, R3, R4: 470Ω, symbol R_Small
- BT1: value Li-Ion 18650 -> LiPo
Connections:
- net GND: now also D1.1 (K), D2.1 (K), D3.1 (K)
- net LED1: now reaches U1.37 (RXD/PIO1_14)
- net LED1: now also R2.1
- net LED2: now reaches U1.38 (MOSI1/PIO1_22)
- net LED2: now also R3.1
- net LED3: now reaches U1.39 (PIO0_15/SWDIO/AD4)
- net LED3: now also R4.1
- new net: D1.2 (A), R2.2
- new net: D2.2 (A), R3.2
- new net: D3.2 (A), R4.2
- no-connect marks 54 -> 51
Other:
- note added: "LEDs"
Changed lines of the file:
@@
 UC-TX
 $Comp
-L GND #PWR10
+L GND #PWR13
 U 1 1 59359076
 P 6250 6300
-F 0 "#PWR10" H 6250 6050 50  0001 C CNN
+F 0 "#PWR13" H 6250 6050 50  0001 C CNN
 F 1 "GND" H 6250 6150 50  0000 C CNN
 F 2 "" H 6250 6300 50  0001 C CNN
@@
 $EndComp
 $Comp
-L GND #PWR7
+L GND #PWR10
 U 1 1 59359351
 P 7650 4150
-F 0 "#PWR7" H 7650 3900 50  0001 C CNN
+F 0 "#PWR10" H 7650 3900 50  0001 C CNN
 F 1 "GND" H 7650 4000 50  0000 C CNN
 F 2 "" H 7650 4150 50  0001 C CNN
@@
 	4200 7300 4200 7400
 $Comp
-L GND #PWR14
+L GND #PWR17
 U 1 1 5935A145
 P 4200 7400
-F 0 "#PWR14" H 4200 7150 50  0001 C CNN
+F 0 "#PWR17" H 4200 7150 50  0001 C CNN
 F 1 "GND" H 4200 7250 50  0000 C CNN
 F 2 "" H 4200 7400 50  0001 C CNN
@@
 $EndComp
 $Comp
-L GND #PWR13
+L GND #PWR16
 U 1 1 5935A165
 P 3900 7400
-F 0 "#PWR13" H 3900 7150 50  0001 C CNN
+F 0 "#PWR16" H 3900 7150 50  0001 C CNN
 F 1 "GND" H 3900 7250 50  0000 C CNN
 F 2 "" H 3900 7400 50  0001 C CNN
@@
 $EndComp
 $Comp
-L GND #PWR11
+L GND #PWR14
 U 1 1 5935A2B3
 P 2400 6700
-F 0 "#PWR11" H 2400 6450 50  0001 C CNN
+F 0 "#PWR14" H 2400 6450 50  0001 C CNN
 F 1 "GND" H 2400 6550 50  0000 C CNN
 F 2 "" H 2400 6700 50  0001 C CNN
@@
 $EndComp
 $Comp
-L GND #PWR12
+L GND #PWR15
 U 1 1 5935A2D3
 P 2600 6700
-F 0 "#PWR12" H 2600 6450 50  0001 C CNN
+F 0 "#PWR15" H 2600 6450 50  0001 C CNN
 F 1 "GND" H 2600 6550 50  0000 C CNN
 F 2 "" H 2600 6700 50  0001 C CNN
@@
 P 750 1350
 F 0 "BT1" H 850 1450 50  0000 L CNN
-F 1 "Li-Ion 18650" V 600 1050 50  0000 L CNN
+F 1 "LiPo" H 850 1350 50  0000 L CNN
 F 2 "" V 750 1410 50  0001 C CNN
 F 3 "" V 750 1410 50  0001 C CNN
@@
 NTRST
 $Comp
-L GND #PWR9
+L GND #PWR12
 U 1 1 59360BFA
 P 10450 4900
-F 0 "#PWR9" H 10450 4650 50  0001 C CNN
+F 0 "#PWR12" H 10450 4650 50  0001 C CNN
 F 1 "GND" H 10450 4750 50  0000 C CNN
 F 2 "" H 10450 4900 50  0001 C CNN
@@
 	9200 4400 9200 4500
 $Comp
-L GND #PWR8
+L GND #PWR11
 U 1 1 59361F74
 P 9200 4500
-F 0 "#PWR8" H 9200 4250 50  0001 C CNN
+F 0 "#PWR11" H 9200 4250 50  0001 C CNN
 F 1 "GND" H 9200 4350 50  0000 C CNN
 F 2 "" H 9200 4500 50  0001 C CNN
@@
 NoConn ~ 1300 4900
 NoConn ~ 1300 5000
-NoConn ~ 1300 5600
 NoConn ~ 1300 5700
 NoConn ~ 1300 5800
@@
 NoConn ~ 3700 5000
 NoConn ~ 3700 4900
-NoConn ~ 3700 4800
 NoConn ~ 3700 4700
 NoConn ~ 3700 4600
@@
 NoConn ~ 3700 4400
 NoConn ~ 3700 4300
-NoConn ~ 3700 4200
 NoConn ~ 3700 4100
 $Comp
@@
 Text GLabel 4800 3750 1    60   Input ~ 0
 3.3V
+Text Notes 5100 1200 0    100  ~ 0
+LEDs
+$Comp
+L R_Small R2
+U 1 1 5973930C
+P 5150 1800
+F 0 "R2" V 5050 1750 50  0000 L CNN
+F 1 "470Ω" V 5250 1800 50  0000 L CNN
+F 2 "" H 5150 1800 50  0001 C CNN
+F 3 "" H 5150 1800 50  0001 C CNN
+	1    5150 1800
+	1    0    0    -1
+$EndComp
+$Comp
+L R_Small R3
+U 1 1 5973935E
+P 5600 1800
+F 0 "R3" V 5500 1750 50  0000 L CNN
+F 1 "470Ω" V 5700 1800 50  0000 L CNN
+F 2 "" H 5600 1800 50  0001 C CNN
+F 3 "" H 5600 1800 50  0001 C CNN
+	1    5600 1800
+	1    0    0    -1
+$EndComp
+$Comp
+L R_Small R4
+U 1 1 597393AA
+P 6050 1800
+F 0 "R4" V 5950 1750 50  0000 L CNN
+F 1 "470Ω" V 6150 1800 50  0000 L CNN
+F 2 "" H 6050 1800 50  0001 C CNN
+F 3 "" H 6050 1800 50  0001 C CNN
+	1    6050 1800
+	1    0    0    -1
+$EndComp
+$Comp
+L LED_Small D1
+U 1 1 59739427
+P 5150 2150
+F 0 "D1" H 5100 2275 50  0000 L CNN
+F 1 "LED" H 5100 2050 50  0000 L CNN
+F 2 "" V 5150 2150 50  0001 C CNN
+F 3 "" V 5150 2150 50  0001 C CNN
+	1    5150 2150
+	0    -1   -1   0
+$EndComp
+$Comp
+L LED_Small D2
+U 1 1 5973949C
+P 5600 2150
+F 0 "D2" H 5550 2275 50  0000 L CNN
+F 1 "LED" H 5550 2050 50  0000 L CNN
+F 2 "" V 5600 2150 50  0001 C CNN
+F 3 "" V 5600 2150 50  0001 C CNN
+	1    5600 2150
+	0    -1   -1   0
+$EndComp
+$Comp
+L LED_Small D3
+U 1 1 5973955C
+P 6050 2150
+F 0 "D3" H 6000 2275 50  0000 L CNN
+F 1 "LED" H 6000 2050 50  0000 L CNN
+F 2 "" V 6050 2150 50  0001 C CNN
+F 3 "" V 6050 2150 50  0001 C CNN
+	1    6050 2150
+	0    -1   -1   0
+$EndComp
+Wire Wire Line
+	5150 2050 5150 1900
+Wire Wire Line
+	5600 1900 5600 2050
+Wire Wire Line
+	6050 2050 6050 1900
+Wire Wire Line
+	5150 2250 5150 2400
+$Comp
+L GND #PWR7
+U 1 1 597398A8
+P 5150 2400
+F 0 "#PWR7" H 5150 2150 50  0001 C CNN
+F 1 "GND" H 5150 2250 50  0000 C CNN
+F 2 "" H 5150 2400 50  0001 C CNN
+F 3 "" H 5150 2400 50  0001 C CNN
+	1    5150 2400
+	1    0    0    -1
+$EndComp
+$Comp
+L GND #PWR8
+U 1 1 597398F6
+P 5600 2400
+F 0 "#PWR8" H 5600 2150 50  0001 C CNN
+F 1 "GND" H 5600 2250 50  0000 C CNN
+F 2 "" H 5600 2400 50  0001 C CNN
+F 3 "" H 5600 2400 50  0001 C CNN
+	1    5600 2400
+	1    0    0    -1
+$EndComp
+$Comp
+L GND #PWR9
+U 1 1 5973993D
+P 6050 2400
+F 0 "#PWR9" H 6050 2150 50  0001 C CNN
+F 1 "GND" H 6050 2250 50  0000 C CNN
+F 2 "" H 6050 2400 50  0001 C CNN
+F 3 "" H 6050 2400 50  0001 C CNN
+	1    6050 2400
+	1    0    0    -1
+$EndComp
+Wire Wire Line
+	6050 2400 6050 2250
+Wire Wire Line
+	5600 2250 5600 2400
+Text GLabel 1300 5600 0    60   Input ~ 0
+LED3
+Text GLabel 3900 4800 2    60   Input ~ 0
+LED2
+Text GLabel 3900 4200 2    60   Input ~ 0
+LED1
+Wire Wire Line
+	3900 4200 3700 4200
+Wire Wire Line
+	3700 4800 3900 4800
+Text GLabel 5150 1550 1    60   Input ~ 0
+LED1
+Text GLabel 5600 1550 1    60   Input ~ 0
+LED2
+Text GLabel 6050 1550 1    60   Input ~ 0
+LED3
+Wire Wire Line
+	5150 1700 5150 1550
+Wire Wire Line
+	5600 1550 5600 1700
+Wire Wire Line
+	6050 1550 6050 1700
 $EndSCHEMATC

Commit message: Add I²C connector and pull-ups
Parts:
- added J?: CONN_01X04, symbol CONN_01X04
- added R? (x2): 10KΩ, symbol R_Small
Connections:
- net 3.3V: now also J?.1 (P1), R?.1, R?.1
- net GND: now also J?.4 (P4)
- net SCL: now also J?.3 (P3), R?.2
- net SDA: now also J?.2 (P2), R?.2
Other:
- note added: "I²C External"
- note added: "I²C Pull-Ups"
- moved on the sheet: U4, U5
Changed lines of the file:
@@
 L SHT21 U4
 U 1 1 5935D012
-P 8250 1850
-F 0 "U4" H 8250 2150 60  0000 C CNN
-F 1 "SHT21" H 8250 1550 60  0000 C CNN
-F 2 "" H 8250 1850 60  0001 C CNN
-F 3 "" H 8250 1850 60  0001 C CNN
-	1    8250 1850
+P 8150 1650
+F 0 "U4" H 8150 1950 60  0000 C CNN
+F 1 "SHT21" H 8150 1350 60  0000 C CNN
+F 2 "" H 8150 1650 60  0001 C CNN
+F 3 "" H 8150 1650 60  0001 C CNN
+	1    8150 1650
 	1    0    0    1
 $EndComp
-Text Notes 7750 1200 0    100  ~ 0
+Text Notes 7350 1050 0    100  ~ 0
 Sensors
-Text GLabel 7750 1850 0    60   Input ~ 0
-3.3V
-Wire Wire Line
-	8750 1850 8850 1850
-Wire Wire Line
-	8850 1850 8850 1950
+Text GLabel 7650 1650 0    60   Input ~ 0
+3.3V
+Wire Wire Line
+	8650 1650 8750 1650
+Wire Wire Line
+	8750 1650 8750 1750
 $Comp
 L GND #PWR5
 U 1 1 5935D6F4
-P 8850 1950
-F 0 "#PWR5" H 8850 1700 50  0001 C CNN
-F 1 "GND" H 8850 1800 50  0000 C CNN
-F 2 "" H 8850 1950 50  0001 C CNN
-F 3 "" H 8850 1950 50  0001 C CNN
-	1    8850 1950
-	1    0    0    -1
-$EndComp
-Text GLabel 7750 1700 0    60   Input ~ 0
+P 8750 1750
+F 0 "#PWR5" H 8750 1500 50  0001 C CNN
+F 1 "GND" H 8750 1600 50  0000 C CNN
+F 2 "" H 8750 1750 50  0001 C CNN
+F 3 "" H 8750 1750 50  0001 C CNN
+	1    8750 1750
+	1    0    0    -1
+$EndComp
+Text GLabel 7650 1500 0    60   Input ~ 0
 SCL
-Text GLabel 8750 1700 2    60   Input ~ 0
+Text GLabel 8650 1500 2    60   Input ~ 0
 SDA
 Text GLabel 1100 4450 0    60   Input ~ 0
@@
 L DS18B20 U5
 U 1 1 5935DFAC
-P 9950 1850
-F 0 "U5" H 9950 1600 60  0000 C CNN
-F 1 "DS18B20" H 9950 2100 60  0000 C CNN
-F 2 "" H 9950 1850 60  0001 C CNN
-F 3 "" H 9950 1850 60  0001 C CNN
-	1    9950 1850
-	1    0    0    -1
-$EndComp
-Text GLabel 10450 1700 2    60   Input ~ 0
-3.3V
-Wire Wire Line
-	10250 1950 10350 1950
-Wire Wire Line
-	10350 1950 10350 2050
+P 9850 1650
+F 0 "U5" H 9850 1400 60  0000 C CNN
+F 1 "DS18B20" H 9850 1900 60  0000 C CNN
+F 2 "" H 9850 1650 60  0001 C CNN
+F 3 "" H 9850 1650 60  0001 C CNN
+	1    9850 1650
+	1    0    0    -1
+$EndComp
+Text GLabel 10350 1500 2    60   Input ~ 0
+3.3V
+Wire Wire Line
+	10150 1750 10250 1750
+Wire Wire Line
+	10250 1750 10250 1850
 $Comp
 L GND #PWR6
 U 1 1 5935E161
-P 10350 2050
-F 0 "#PWR6" H 10350 1800 50  0001 C CNN
-F 1 "GND" H 10350 1900 50  0000 C CNN
-F 2 "" H 10350 2050 50  0001 C CNN
-F 3 "" H 10350 2050 50  0001 C CNN
-	1    10350 2050
-	1    0    0    -1
-$EndComp
-Wire Wire Line
-	10450 1700 10350 1700
-Wire Wire Line
-	10350 1700 10350 1750
-Wire Wire Line
-	10350 1750 10250 1750
-Wire Wire Line
-	10250 1850 10350 1850
-Wire Wire Line
-	10350 1850 10350 1900
-Wire Wire Line
-	10350 1900 10450 1900
-Text GLabel 10450 1900 2    60   Input ~ 0
+P 10250 1850
+F 0 "#PWR6" H 10250 1600 50  0001 C CNN
+F 1 "GND" H 10250 1700 50  0000 C CNN
+F 2 "" H 10250 1850 50  0001 C CNN
+F 3 "" H 10250 1850 50  0001 C CNN
+	1    10250 1850
+	1    0    0    -1
+$EndComp
+Wire Wire Line
+	10350 1500 10250 1500
+Wire Wire Line
+	10250 1500 10250 1550
+Wire Wire Line
+	10250 1550 10150 1550
+Wire Wire Line
+	10150 1650 10250 1650
+Wire Wire Line
+	10250 1650 10250 1700
+Wire Wire Line
+	10250 1700 10350 1700
+Text GLabel 10350 1700 2    60   Input ~ 0
 DS18B20
 Wire Wire Line
@@
 Wire Wire Line
 	6050 1550 6050 1700
+$Comp
+L R_Small R?
+U 1 1 5973BD8F
+P 7950 2750
+F 0 "R?" V 7850 2700 50  0000 L CNN
+F 1 "10KΩ" V 8050 2650 50  0000 L CNN
+F 2 "" H 7950 2750 50  0001 C CNN
+F 3 "" H 7950 2750 50  0001 C CNN
+	1    7950 2750
+	0    1    1    0
+$EndComp
+Text GLabel 7750 2750 0    60   Input ~ 0
+SCL
+Wire Wire Line
+	7750 2750 7850 2750
+Wire Wire Line
+	8050 2750 8150 2750
+Text GLabel 8150 2750 2    60   Input ~ 0
+3.3V
+$Comp
+L R_Small R?
+U 1 1 5973C254
+P 7950 3100
+F 0 "R?" V 7850 3050 50  0000 L CNN
+F 1 "10KΩ" V 8050 3000 50  0000 L CNN
+F 2 "" H 7950 3100 50  0001 C CNN
+F 3 "" H 7950 3100 50  0001 C CNN
+	1    7950 3100
+	0    1    1    0
+$EndComp
+Text GLabel 7750 3100 0    60   Input ~ 0
+SDA
+Wire Wire Line
+	7750 3100 7850 3100
+Wire Wire Line
+	8050 3100 8150 3100
+Text GLabel 8150 3100 2    60   Input ~ 0
+3.3V
+Text Notes 7500 2500 0    100  ~ 0
+I²C Pull-Ups
+$Comp
+L CONN_01X04 J?
+U 1 1 5973C740
+P 10250 2800
+F 0 "J?" H 10250 3050 50  0000 C CNN
+F 1 "CONN_01X04" V 10350 2800 50  0000 C CNN
+F 2 "" H 10250 2800 50  0001 C CNN
+F 3 "" H 10250 2800 50  0001 C CNN
+	1    10250 2800
+	1    0    0    -1
+$EndComp
+Text Notes 9450 2400 0    100  ~ 0
+I²C External
+Text GLabel 9950 2650 0    60   Input ~ 0
+3.3V
+Wire Wire Line
+	9950 2650 10050 2650
+Wire Wire Line
+	10050 2950 9950 2950
+Wire Wire Line
+	9950 2950 9950 3050
+$Comp
+L GND #PWR?
+U 1 1 5973CA0A
+P 9950 3050
+F 0 "#PWR?" H 9950 2800 50  0001 C CNN
+F 1 "GND" H 9950 2900 50  0000 C CNN
+F 2 "" H 9950 3050 50  0001 C CNN
+F 3 "" H 9950 3050 50  0001 C CNN
+	1    9950 3050
+	1    0    0    -1
+$EndComp
+Text GLabel 9650 2750 0    60   Input ~ 0
+SDA
+Text GLabel 9950 2850 0    60   Input ~ 0
+SCL
+Wire Wire Line
+	9650 2750 10050 2750
+Wire Wire Line
+	9950 2850 10050 2850
 $EndSCHEMATC

Commit message: Add UART debug pins
Parts:
- added J?: CONN_01X02, symbol CONN_01X02
- added J?: CONN_01X01, symbol CONN_01X01
Connections:
- net LED1: now also U1.38 (MOSI1/PIO1_22); no longer U1.37 (RXD/PIO1_14)
- net LED2: now also U1.39 (PIO0_15/SWDIO/AD4); no longer U1.38 (MOSI1/PIO1_22)
- net LED3: now also U1.45 (PIO0_17/CT32B0_C0/SCLK); no longer U1.39 (PIO0_15/SWDIO/AD4)
- net UC-TX1: now reaches U1.36 (TXD/PIO1_13)
- net UC-TX1: now also J?.2 (P2)
- net UC-RX renamed UC-RX0
- net UC-TX renamed UC-TX0
- net UC-TX0: now also J?.1 (P1)
- new net UC-RX1: J?.1 (P1), U1.37 (RXD/PIO1_14)
- no-connect marks 51 -> 49
Other:
- note added: "UART"
Changed lines of the file:
@@
 $EndDescr
-$Comp
-L LPC11U24FBD48 U1
-U 1 1 59356CC0
-P 2500 5400
-F 0 "U1" H 1450 6850 50  0000 C CNN
-F 1 "LPC11U24FBD48" H 1700 4180 50  0000 C CNN
-F 2 "Housings_QFP:LQFP-48_7x7mm_Pitch0.5mm" H 3450 4200 50  0001 C CNN
-F 3 "" H 2500 3925 50  0001 C CNN
-	1    2500 5400
-	1    0    0    -1
-$EndComp
 $Comp
 L RN2483 U3
@@
 $EndComp
 Text GLabel 1100 5850 0    60   Input ~ 0
-UC-RX
+UC-RX0
 Text GLabel 1100 6050 0    60   Input ~ 0
-UC-TX
+UC-TX0
 Text GLabel 7350 5500 2    60   Input ~ 0
-UC-RX
+UC-RX0
 Text GLabel 7350 5300 2    60   Input ~ 0
-UC-TX
+UC-TX0
 $Comp
 L GND #PWR13
@@
 NoConn ~ 1300 5000
 NoConn ~ 1300 5700
-NoConn ~ 1300 5800
 NoConn ~ 1300 6100
 NoConn ~ 1300 6200
@@
 NoConn ~ 3700 4400
 NoConn ~ 3700 4300
-NoConn ~ 3700 4100
 $Comp
 L R R1
@@
 	5600 2250 5600 2400
 Text GLabel 1300 5600 0    60   Input ~ 0
+LED2
+Text GLabel 3900 4800 2    60   Input ~ 0
+LED1
+Text GLabel 950  5700 0    60   Input ~ 0
 LED3
-Text GLabel 3900 4800 2    60   Input ~ 0
-LED2
-Text GLabel 3900 4200 2    60   Input ~ 0
-LED1
-Wire Wire Line
-	3900 4200 3700 4200
 Wire Wire Line
 	3700 4800 3900 4800
@@
 Wire Wire Line
 	9950 2850 10050 2850
+$Comp
+L CONN_01X02 J?
+U 1 1 5973D2E1
+P 4100 2450
+F 0 "J?" H 4100 2600 50  0000 C CNN
+F 1 "CONN_01X02" V 4200 2450 50  0000 C CNN
+F 2 "" H 4100 2450 50  0001 C CNN
+F 3 "" H 4100 2450 50  0001 C CNN
+	1    4100 2450
+	1    0    0    -1
+$EndComp
+Text Notes 3300 2150 0    100  ~ 0
+UART
+Wire Wire Line
+	950  5700 1250 5700
+Wire Wire Line
+	1250 5700 1250 5800
+Wire Wire Line
+	1250 5800 1300 5800
+$Comp
+L LPC11U24FBD48 U1
+U 1 1 59356CC0
+P 2500 5400
+F 0 "U1" H 1450 6850 50  0000 C CNN
+F 1 "LPC11U24FBD48" H 1700 4180 50  0000 C CNN
+F 2 "Housings_QFP:LQFP-48_7x7mm_Pitch0.5mm" H 3450 4200 50  0001 C CNN
+F 3 "" H 2500 3925 50  0001 C CNN
+	1    2500 5400
+	1    0    0    -1
+$EndComp
+Text GLabel 3900 4100 2    60   Input ~ 0
+UC-TX1
+Text GLabel 3900 4200 2    60   Input ~ 0
+UC-RX1
+Wire Wire Line
+	3900 4100 3700 4100
+Wire Wire Line
+	3700 4200 3900 4200
+Text GLabel 3750 2400 0    60   Input ~ 0
+UC-RX1
+Text GLabel 3750 2500 0    60   Input ~ 0
+UC-TX1
+Wire Wire Line
+	3750 2400 3900 2400
+Wire Wire Line
+	3900 2500 3750 2500
+$Comp
+L CONN_01X01 J?
+U 1 1 5973F46D
+P 4100 3050
+F 0 "J?" H 4100 3150 50  0000 C CNN
+F 1 "CONN_01X01" V 4200 3050 50  0000 C CNN
+F 2 "" H 4100 3050 50  0001 C CNN
+F 3 "" H 4100 3050 50  0001 C CNN
+	1    4100 3050
+	1    0    0    -1
+$EndComp
+Wire Wire Line
+	3900 3050 3750 3050
+Text GLabel 3750 3050 0    60   Input ~ 0
+UC-TX0
 $EndSCHEMATC
