File: pcb/watertemp_v1.sch (KiCad schematic (older format))
At the start: 27 parts, among them J1 RN2483 Ext, J2 SWD, J3 CONN_01X04, J4 UART1, J5 UART2, U1 LPC11U24FBD48, U2 RN2483, U3 SHT21, U4 LP5907-Q1, U5 DS18B20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

Commit message: Continue work on PCB
Parts:
- added C5: 100nF, Capacitors_SMD:C_0805, symbol C_Small
- added R8: 4.7K, Resistors_SMD:R_0805_HandSoldering, symbol R_Small
- BT1: value LiPo -> LiIo; footprint Connectors_JST:JST_PH_B2B-PH-SM4-TB_02x2.00mm_Straight -> Battery_Clips:36-54-ND; Digikey 455-1734-1-ND -> 36-54-ND
- J3: value CONN_01X04 -> I2C
- R4, R5, R6, R7: footprint Resistors_SMD:R_1206_HandSoldering -> Resistors_SMD:R_0805_HandSoldering
- Y1: footprint Crystals:Crystal_SMD_5032-2pin_5.0x3.2mm -> Crystals:Crystal_SMD_Abracon_ABM8G-4pin_3.2x2.5mm; Digikey CTX1435CT-ND -> 535-10901-1-ND; Part CTS 445C35A12M00000 -> ABM8G-12.000MHZ-4Y-T3
Connections:
- net 3.3V: now also C5.2, R8.1
- net DS18B20: now also R8.2
- net GND: now also C5.1
Changed lines of the file:
@@
 UC-TX0
 $Comp
-L GND #PWR01
+L GND #PWR1
 U 1 1 59359076
 P 2250 7500
-F 0 "#PWR01" H 2250 7250 50  0001 C CNN
+F 0 "#PWR1" H 2250 7250 50  0001 C CNN
 F 1 "GND" H 2250 7350 50  0000 C CNN
 F 2 "" H 2250 7500 50  0001 C CNN
@@
 $EndComp
 $Comp
-L GND #PWR02
+L GND #PWR4
 U 1 1 59359351
 P 3650 5350
-F 0 "#PWR02" H 3650 5100 50  0001 C CNN
+F 0 "#PWR4" H 3650 5100 50  0001 C CNN
 F 1 "GND" H 3650 5200 50  0000 C CNN
 F 2 "" H 3650 5350 50  0001 C CNN
@@
 F 0 "Y1" H 4000 4000 50  0000 C CNN
 F 1 "12MHz" H 4000 3700 50  0000 C CNN
-F 2 "Crystals:Crystal_SMD_5032-2pin_5.0x3.2mm" H 4000 3850 50  0001 C CNN
+F 2 "Crystals:Crystal_SMD_Abracon_ABM8G-4pin_3.2x2.5mm" H 4000 3850 50  0001 C CNN
 F 3 "" H 4000 3850 50  0001 C CNN
-F 4 "CTS 445C35A12M00000" H 4000 3850 60  0001 C CNN "Part"
-F 5 "CTX1435CT-ND" H 4000 3850 60  0001 C CNN "Digikey"
+F 4 "ABM8G-12.000MHZ-4Y-T3" H 4000 3850 60  0001 C CNN "Part"
+F 5 "535-10901-1-ND" H 4000 3850 60  0001 C CNN "Digikey"
 	1    4000 3850
 	-1   0    0    1
@@
 	4150 4350 4150 4450
 $Comp
-L GND #PWR03
+L GND #PWR6
 U 1 1 5935A145
 P 4150 4450
-F 0 "#PWR03" H 4150 4200 50  0001 C CNN
+F 0 "#PWR6" H 4150 4200 50  0001 C CNN
 F 1 "GND" H 4150 4300 50  0000 C CNN
 F 2 "" H 4150 4450 50  0001 C CNN
@@
 $EndComp
 $Comp
-L GND #PWR04
+L GND #PWR5
 U 1 1 5935A165
 P 3850 4450
-F 0 "#PWR04" H 3850 4200 50  0001 C CNN
+F 0 "#PWR5" H 3850 4200 50  0001 C CNN
 F 1 "GND" H 3850 4300 50  0000 C CNN
 F 2 "" H 3850 4450 50  0001 C CNN
@@
 $EndComp
 $Comp
-L GND #PWR05
+L GND #PWR2
 U 1 1 5935A2B3
 P 2350 3750
-F 0 "#PWR05" H 2350 3500 50  0001 C CNN
+F 0 "#PWR2" H 2350 3500 50  0001 C CNN
 F 1 "GND" H 2350 3600 50  0000 C CNN
 F 2 "" H 2350 3750 50  0001 C CNN
@@
 $EndComp
 $Comp
-L GND #PWR06
+L GND #PWR3
 U 1 1 5935A2D3
 P 2550 3750
-F 0 "#PWR06" H 2550 3500 50  0001 C CNN
+F 0 "#PWR3" H 2550 3500 50  0001 C CNN
 F 1 "GND" H 2550 3600 50  0000 C CNN
 F 2 "" H 2550 3750 50  0001 C CNN
@@
 P 5100 1650
 F 0 "BT1" H 5200 1750 50  0000 L CNN
-F 1 "LiPo" H 5200 1650 50  0000 L CNN
-F 2 "Connectors_JST:JST_PH_B2B-PH-SM4-TB_02x2.00mm_Straight" V 5100 1710 50  0001 C CNN
+F 1 "LiIo" H 5200 1650 50  0000 L CNN
+F 2 "Battery_Clips:36-54-ND" V 5100 1710 50  0001 C CNN
 F 3 "" V 5100 1710 50  0001 C CNN
-F 4 "455-1734-1-ND" H 5100 1650 60  0001 C CNN "Digikey"
+F 4 "36-54-ND" H 5100 1650 60  0001 C CNN "Digikey"
 	1    5100 1650
 	1    0    0    -1
@@
 NoConn ~ 5900 1600
 $Comp
-L GND #PWR07
+L GND #PWR7
 U 1 1 5935BDCA
 P 5100 1850
-F 0 "#PWR07" H 5100 1600 50  0001 C CNN
+F 0 "#PWR7" H 5100 1600 50  0001 C CNN
 F 1 "GND" H 5100 1700 50  0000 C CNN
 F 2 "" H 5100 1850 50  0001 C CNN
@@
 3.3V
 $Comp
-L GND #PWR08
+L GND #PWR11
 U 1 1 5935BF9C
 P 6800 1600
-F 0 "#PWR08" H 6800 1350 50  0001 C CNN
+F 0 "#PWR11" H 6800 1350 50  0001 C CNN
 F 1 "GND" H 6800 1450 50  0000 C CNN
 F 2 "" H 6800 1600 50  0001 C CNN
@@
 	5600 1800 5600 1900
 $Comp
-L GND #PWR09
+L GND #PWR8
 U 1 1 5935C646
 P 5600 1900
-F 0 "#PWR09" H 5600 1650 50  0001 C CNN
+F 0 "#PWR8" H 5600 1650 50  0001 C CNN
 F 1 "GND" H 5600 1750 50  0000 C CNN
 F 2 "" H 5600 1900 50  0001 C CNN
@@
 	7100 1800 7100 1900
 $Comp
-L GND #PWR010
+L GND #PWR12
 U 1 1 5935C857
 P 7100 1900
-F 0 "#PWR010" H 7100 1650 50  0001 C CNN
+F 0 "#PWR12" H 7100 1650 50  0001 C CNN
 F 1 "GND" H 7100 1750 50  0000 C CNN
 F 2 "" H 7100 1900 50  0001 C CNN
@@
 Text Notes 5050 2900 0    100  ~ 0
 Sensors
-Text GLabel 5300 3350 0    60   Input ~ 0
+Text GLabel 5200 3350 0    60   Input ~ 0
 3.3V
 Wire Wire Line
@@
 	6400 3350 6400 3450
 $Comp
-L GND #PWR011
+L GND #PWR10
 U 1 1 5935D6F4
 P 6400 3450
-F 0 "#PWR011" H 6400 3200 50  0001 C CNN
+F 0 "#PWR10" H 6400 3200 50  0001 C CNN
 F 1 "GND" H 6400 3300 50  0000 C CNN
 F 2 "" H 6400 3450 50  0001 C CNN
@@
 	1    0    0    -1
 $EndComp
-Text GLabel 5300 3200 0    60   Input ~ 0
+Text GLabel 5200 3200 0    60   Input ~ 0
 SCL
-Text GLabel 6300 3200 2    60   Input ~ 0
+Text GLabel 6400 3200 2    60   Input ~ 0
 SDA
 Text GLabel 1050 1500 0    60   Input ~ 0
@@
 	1    0    0    -1
 $EndComp
-Text GLabel 7550 3200 2    60   Input ~ 0
+Text GLabel 7700 3100 2    60   Input ~ 0
 3.3V
 Wire Wire Line
@@
 	7450 3450 7450 3550
 $Comp
-L GND #PWR012
+L GND #PWR13
 U 1 1 5935E161
 P 7450 3550
-F 0 "#PWR012" H 7450 3300 50  0001 C CNN
+F 0 "#PWR13" H 7450 3300 50  0001 C CNN
 F 1 "GND" H 7450 3400 50  0000 C CNN
 F 2 "" H 7450 3550 50  0001 C CNN
@@
 $EndComp
 Wire Wire Line
-	7550 3200 7450 3200
-Wire Wire Line
-	7450 3200 7450 3250
+	7450 3100 7700 3100
+Wire Wire Line
+	7450 3100 7450 3250
 Wire Wire Line
 	7450 3250 7350 3250
@@
 	7450 3350 7450 3400
 Wire Wire Line
-	7450 3400 7550 3400
-Text GLabel 7550 3400 2    60   Input ~ 0
+	7450 3400 7700 3400
+Text GLabel 7700 3400 2    60   Input ~ 0
 DS18B20
 Wire Wire Line
@@
 DS18B20
 $Comp
-L PWR_FLAG #FLG013
+L PWR_FLAG #FLG1
 U 1 1 5936016C
 P 5300 1350
-F 0 "#FLG013" H 5300 1425 50  0001 C CNN
+F 0 "#FLG1" H 5300 1425 50  0001 C CNN
 F 1 "PWR_FLAG" H 5300 1500 50  0000 C CNN
 F 2 "" H 5300 1350 50  0001 C CNN
@@
 F 0 "R5" V 880 5200 50  0000 C CNN
 F 1 "10KΩ" V 700 5200 50  0000 C CNN
-F 2 "Resistors_SMD:R_1206_HandSoldering" V 730 5200 50  0001 C CNN
+F 2 "Resistors_SMD:R_0805_HandSoldering" V 730 5200 50  0001 C CNN
 F 3 "" H 800 5200 50  0001 C CNN
 	1    800  5200
@@
 	9250 1950 9250 2100
 $Comp
-L GND #PWR014
+L GND #PWR15
 U 1 1 597398A8
 P 9250 2100
-F 0 "#PWR014" H 9250 1850 50  0001 C CNN
+F 0 "#PWR15" H 9250 1850 50  0001 C CNN
 F 1 "GND" H 9250 1950 50  0000 C CNN
 F 2 "" H 9250 2100 50  0001 C CNN
@@
 $EndComp
 $Comp
-L GND #PWR015
+L GND #PWR16
 U 1 1 597398F6
 P 9700 2100
-F 0 "#PWR015" H 9700 1850 50  0001 C CNN
+F 0 "#PWR16" H 9700 1850 50  0001 C CNN
 F 1 "GND" H 9700 1950 50  0000 C CNN
 F 2 "" H 9700 2100 50  0001 C CNN
@@
 $EndComp
 $Comp
-L GND #PWR016
+L GND #PWR18
 U 1 1 5973993D
 P 10150 2100
-F 0 "#PWR016" H 10150 1850 50  0001 C CNN
+F 0 "#PWR18" H 10150 1850 50  0001 C CNN
 F 1 "GND" H 10150 1950 50  0000 C CNN
 F 2 "" H 10150 2100 50  0001 C CNN
@@
 F 0 "R6" V 5450 4900 50  0000 L CNN
 F 1 "10KΩ" V 5650 4850 50  0000 L CNN
-F 2 "Resistors_SMD:R_1206_HandSoldering" H 5550 4950 50  0001 C CNN
+F 2 "Resistors_SMD:R_0805_HandSoldering" H 5550 4950 50  0001 C CNN
 F 3 "" H 5550 4950 50  0001 C CNN
 	1    5550 4950
@@
 F 0 "R7" V 5450 5250 50  0000 L CNN
 F 1 "10KΩ" V 5650 5200 50  0000 L CNN
-F 2 "Resistors_SMD:R_1206_HandSoldering" H 5550 5300 50  0001 C CNN
+F 2 "Resistors_SMD:R_0805_HandSoldering" H 5550 5300 50  0001 C CNN
 F 3 "" H 5550 5300 50  0001 C CNN
 	1    5550 5300
@@
 P 7850 5100
 F 0 "J3" H 7850 5350 50  0000 C CNN
-F 1 "CONN_01X04" V 7950 5100 50  0000 C CNN
+F 1 "I2C" V 7950 5100 50  0000 C CNN
 F 2 "Pin_Headers:Pin_Header_Straight_1x04_Pitch2.54mm" H 7850 5100 50  0001 C CNN
 F 3 "" H 7850 5100 50  0001 C CNN
@@
 	7550 5250 7550 5350
 $Comp
-L GND #PWR017
+L GND #PWR14
 U 1 1 5973CA0A
 P 7550 5350
-F 0 "#PWR017" H 7550 5100 50  0001 C CNN
+F 0 "#PWR14" H 7550 5100 50  0001 C CNN
 F 1 "GND" H 7550 5200 50  0000 C CNN
 F 2 "" H 7550 5350 50  0001 C CNN
@@
 	5750 7300 5750 7400
 $Comp
-L GND #PWR018
+L GND #PWR9
 U 1 1 597403FE
 P 5750 7400
-F 0 "#PWR018" H 5750 7150 50  0001 C CNN
+F 0 "#PWR9" H 5750 7150 50  0001 C CNN
 F 1 "GND" H 5750 7250 50  0000 C CNN
 F 2 "" H 5750 7400 50  0001 C CNN
@@
 	9750 3400 9750 3900
 $Comp
-L GND #PWR019
+L GND #PWR17
 U 1 1 59753E6C
 P 9750 3900
-F 0 "#PWR019" H 9750 3650 50  0001 C CNN
+F 0 "#PWR17" H 9750 3650 50  0001 C CNN
 F 1 "GND" H 9750 3750 50  0000 C CNN
 F 2 "" H 9750 3900 50  0001 C CNN
@@
 F 0 "R4" V 730 1000 50  0000 C CNN
 F 1 "10KΩ" V 550 1000 50  0000 C CNN
-F 2 "Resistors_SMD:R_1206_HandSoldering" V 580 1000 50  0001 C CNN
+F 2 "Resistors_SMD:R_0805_HandSoldering" V 580 1000 50  0001 C CNN
 F 3 "" H 650 1000 50  0001 C CNN
 	1    650  1000
@@
 Wire Wire Line
 	9600 5950 9750 5950
+$Comp
+L R_Small R8
+U 1 1 59922965
+P 7650 3250
+F 0 "R8" V 7650 3200 50  0000 L CNN
+F 1 "4.7K" H 7700 3250 50  0000 L CNN
+F 2 "Resistors_SMD:R_0805_HandSoldering" H 7650 3250 50  0001 C CNN
+F 3 "" H 7650 3250 50  0001 C CNN
+	1    7650 3250
+	1    0    0    -1
+$EndComp
+Wire Wire Line
+	7650 3150 7650 3100
+Connection ~ 7650 3100
+Wire Wire Line
+	7650 3350 7650 3400
+Connection ~ 7650 3400
+$Comp
+L C_Small C5
+U 1 1 599223DA
+P 5800 3850
+F 0 "C5" H 5810 3920 50  0000 L CNN
+F 1 "100nF" H 5810 3770 50  0000 L CNN
+F 2 "Capacitors_SMD:C_0805" H 5800 3850 50  0001 C CNN
+F 3 "" H 5800 3850 50  0001 C CNN
+	1    5800 3850
+	0    1    1    0
+$EndComp
+Wire Wire Line
+	5900 3850 6300 3850
+Wire Wire Line
+	6300 3850 6300 3350
+Wire Wire Line
+	5700 3850 5300 3850
+Wire Wire Line
+	5300 3850 5300 3350
+Wire Wire Line
+	5300 3350 5200 3350
+Wire Wire Line
+	5200 3200 5300 3200
+Wire Wire Line
+	6400 3200 6300 3200
 $EndSCHEMATC

Commit message: Finish routing first version
Parts:
- added C6, C7: 100nF, Capacitors_SMD:C_0805, symbol C_Small
- R1, R2, R3, R4, R5, R6, R7: footprint Resistors_SMD:R_0805_HandSoldering -> Resistors_SMD:R_0805
- U1: Digikey (none) -> 568-8460-ND
Connections:
- net 3.3V: now also C6.1, C7.2
- net GND: now also C6.2, C7.1
Changed lines of the file:
@@
 UC-TX0
 $Comp
-L GND #PWR1
+L GND #PWR01
 U 1 1 59359076
 P 2250 7500
-F 0 "#PWR1" H 2250 7250 50  0001 C CNN
+F 0 "#PWR01" H 2250 7250 50  0001 C CNN
 F 1 "GND" H 2250 7350 50  0000 C CNN
 F 2 "" H 2250 7500 50  0001 C CNN
@@
 $EndComp
 $Comp
-L GND #PWR4
+L GND #PWR02
 U 1 1 59359351
 P 3650 5350
-F 0 "#PWR4" H 3650 5100 50  0001 C CNN
+F 0 "#PWR02" H 3650 5100 50  0001 C CNN
 F 1 "GND" H 3650 5200 50  0000 C CNN
 F 2 "" H 3650 5350 50  0001 C CNN
@@
 	4150 4350 4150 4450
 $Comp
-L GND #PWR6
+L GND #PWR03
 U 1 1 5935A145
 P 4150 4450
-F 0 "#PWR6" H 4150 4200 50  0001 C CNN
+F 0 "#PWR03" H 4150 4200 50  0001 C CNN
 F 1 "GND" H 4150 4300 50  0000 C CNN
 F 2 "" H 4150 4450 50  0001 C CNN
@@
 $EndComp
 $Comp
-L GND #PWR5
+L GND #PWR04
 U 1 1 5935A165
 P 3850 4450
-F 0 "#PWR5" H 3850 4200 50  0001 C CNN
+F 0 "#PWR04" H 3850 4200 50  0001 C CNN
 F 1 "GND" H 3850 4300 50  0000 C CNN
 F 2 "" H 3850 4450 50  0001 C CNN
@@
 $EndComp
 $Comp
-L GND #PWR2
+L GND #PWR05
 U 1 1 5935A2B3
 P 2350 3750
-F 0 "#PWR2" H 2350 3500 50  0001 C CNN
+F 0 "#PWR05" H 2350 3500 50  0001 C CNN
 F 1 "GND" H 2350 3600 50  0000 C CNN
 F 2 "" H 2350 3750 50  0001 C CNN
@@
 $EndComp
 $Comp
-L GND #PWR3
+L GND #PWR06
 U 1 1 5935A2D3
 P 2550 3750
-F 0 "#PWR3" H 2550 3500 50  0001 C CNN
+F 0 "#PWR06" H 2550 3500 50  0001 C CNN
 F 1 "GND" H 2550 3600 50  0000 C CNN
 F 2 "" H 2550 3750 50  0001 C CNN
@@
 NoConn ~ 5900 1600
 $Comp
-L GND #PWR7
+L GND #PWR07
 U 1 1 5935BDCA
 P 5100 1850
-F 0 "#PWR7" H 5100 1600 50  0001 C CNN
+F 0 "#PWR07" H 5100 1600 50  0001 C CNN
 F 1 "GND" H 5100 1700 50  0000 C CNN
 F 2 "" H 5100 1850 50  0001 C CNN
@@
 3.3V
 $Comp
-L GND #PWR11
+L GND #PWR08
 U 1 1 5935BF9C
 P 6800 1600
-F 0 "#PWR11" H 6800 1350 50  0001 C CNN
+F 0 "#PWR08" H 6800 1350 50  0001 C CNN
 F 1 "GND" H 6800 1450 50  0000 C CNN
 F 2 "" H 6800 1600 50  0001 C CNN
@@
 	5600 1800 5600 1900
 $Comp
-L GND #PWR8
+L GND #PWR09
 U 1 1 5935C646
 P 5600 1900
-F 0 "#PWR8" H 5600 1650 50  0001 C CNN
+F 0 "#PWR09" H 5600 1650 50  0001 C CNN
 F 1 "GND" H 5600 1750 50  0000 C CNN
 F 2 "" H 5600 1900 50  0001 C CNN
@@
 	7100 1800 7100 1900
 $Comp
-L GND #PWR12
+L GND #PWR010
 U 1 1 5935C857
 P 7100 1900
-F 0 "#PWR12" H 7100 1650 50  0001 C CNN
+F 0 "#PWR010" H 7100 1650 50  0001 C CNN
 F 1 "GND" H 7100 1750 50  0000 C CNN
 F 2 "" H 7100 1900 50  0001 C CNN
@@
 	7100 1500 7100 1400
 Connection ~ 7100 1400
-Text GLabel 2350 950  1    60   Input ~ 0
-3.3V
-Text GLabel 2550 950  1    60   Input ~ 0
+Text GLabel 2350 800  1    60   Input ~ 0
+3.3V
+Text GLabel 2550 800  1    60   Input ~ 0
 3.3V
 NoConn ~ 3650 2950
@@
 	6400 3350 6400 3450
 $Comp
-L GND #PWR10
+L GND #PWR011
 U 1 1 5935D6F4
 P 6400 3450
-F 0 "#PWR10" H 6400 3200 50  0001 C CNN
+F 0 "#PWR011" H 6400 3200 50  0001 C CNN
 F 1 "GND" H 6400 3300 50  0000 C CNN
 F 2 "" H 6400 3450 50  0001 C CNN
@@
 	7450 3450 7450 3550
 $Comp
-L GND #PWR13
+L GND #PWR012
 U 1 1 5935E161
 P 7450 3550
-F 0 "#PWR13" H 7450 3300 50  0001 C CNN
+F 0 "#PWR012" H 7450 3300 50  0001 C CNN
 F 1 "GND" H 7450 3400 50  0000 C CNN
 F 2 "" H 7450 3550 50  0001 C CNN
@@
 DS18B20
 $Comp
-L PWR_FLAG #FLG1
+L PWR_FLAG #FLG013
 U 1 1 5936016C
 P 5300 1350
-F 0 "#FLG1" H 5300 1425 50  0001 C CNN
+F 0 "#FLG013" H 5300 1425 50  0001 C CNN
 F 1 "PWR_FLAG" H 5300 1500 50  0000 C CNN
 F 2 "" H 5300 1350 50  0001 C CNN
@@
 F 0 "R5" V 880 5200 50  0000 C CNN
 F 1 "10KΩ" V 700 5200 50  0000 C CNN
-F 2 "Resistors_SMD:R_0805_HandSoldering" V 730 5200 50  0001 C CNN
+F 2 "Resistors_SMD:R_0805" V 730 5200 50  0001 C CNN
 F 3 "" H 800 5200 50  0001 C CNN
 	1    800  5200
@@
 F 0 "R1" V 9150 1450 50  0000 L CNN
 F 1 "470Ω" V 9350 1500 50  0000 L CNN
-F 2 "Resistors_SMD:R_0805_HandSoldering" H 9250 1500 50  0001 C CNN
+F 2 "Resistors_SMD:R_0805" H 9250 1500 50  0001 C CNN
 F 3 "" H 9250 1500 50  0001 C CNN
 	1    9250 1500
@@
 F 0 "R2" V 9600 1450 50  0000 L CNN
 F 1 "470Ω" V 9800 1500 50  0000 L CNN
-F 2 "Resistors_SMD:R_0805_HandSoldering" H 9700 1500 50  0001 C CNN
+F 2 "Resistors_SMD:R_0805" H 9700 1500 50  0001 C CNN
 F 3 "" H 9700 1500 50  0001 C CNN
 	1    9700 1500
@@
 F 0 "R3" V 10050 1450 50  0000 L CNN
 F 1 "470Ω" V 10250 1500 50  0000 L CNN
-F 2 "Resistors_SMD:R_0805_HandSoldering" H 10150 1500 50  0001 C CNN
+F 2 "Resistors_SMD:R_0805" H 10150 1500 50  0001 C CNN
 F 3 "" H 10150 1500 50  0001 C CNN
 	1    10150 1500
@@
 	9250 1950 9250 2100
 $Comp
-L GND #PWR15
+L GND #PWR014
 U 1 1 597398A8
 P 9250 2100
-F 0 "#PWR15" H 9250 1850 50  0001 C CNN
+F 0 "#PWR014" H 9250 1850 50  0001 C CNN
 F 1 "GND" H 9250 1950 50  0000 C CNN
 F 2 "" H 9250 2100 50  0001 C CNN
@@
 $EndComp
 $Comp
-L GND #PWR16
+L GND #PWR015
 U 1 1 597398F6
 P 9700 2100
-F 0 "#PWR16" H 9700 1850 50  0001 C CNN
+F 0 "#PWR015" H 9700 1850 50  0001 C CNN
 F 1 "GND" H 9700 1950 50  0000 C CNN
 F 2 "" H 9700 2100 50  0001 C CNN
@@
 $EndComp
 $Comp
-L GND #PWR18
+L GND #PWR016
 U 1 1 5973993D
 P 10150 2100
-F 0 "#PWR18" H 10150 1850 50  0001 C CNN
+F 0 "#PWR016" H 10150 1850 50  0001 C CNN
 F 1 "GND" H 10150 1950 50  0000 C CNN
 F 2 "" H 10150 2100 50  0001 C CNN
@@
 F 0 "R6" V 5450 4900 50  0000 L CNN
 F 1 "10KΩ" V 5650 4850 50  0000 L CNN
-F 2 "Resistors_SMD:R_0805_HandSoldering" H 5550 4950 50  0001 C CNN
+F 2 "Resistors_SMD:R_0805" H 5550 4950 50  0001 C CNN
 F 3 "" H 5550 4950 50  0001 C CNN
 	1    5550 4950
@@
 F 0 "R7" V 5450 5250 50  0000 L CNN
 F 1 "10KΩ" V 5650 5200 50  0000 L CNN
-F 2 "Resistors_SMD:R_0805_HandSoldering" H 5550 5300 50  0001 C CNN
+F 2 "Resistors_SMD:R_0805" H 5550 5300 50  0001 C CNN
 F 3 "" H 5550 5300 50  0001 C CNN
 	1    5550 5300
@@
 	7550 5250 7550 5350
 $Comp
-L GND #PWR14
+L GND #PWR017
 U 1 1 5973CA0A
 P 7550 5350
-F 0 "#PWR14" H 7550 5100 50  0001 C CNN
+F 0 "#PWR017" H 7550 5100 50  0001 C CNN
 F 1 "GND" H 7550 5200 50  0000 C CNN
 F 2 "" H 7550 5350 50  0001 C CNN
@@
 F 2 "Housings_QFP:LQFP-48_7x7mm_Pitch0.5mm" H 3400 1250 50  0001 C CNN
 F 3 "" H 2450 975 50  0001 C CNN
+F 4 "568-8460-ND" H 2450 2450 60  0001 C CNN "Digikey"
 	1    2450 2450
 	1    0    0    -1
@@
 	5750 7300 5750 7400
 $Comp
-L GND #PWR9
+L GND #PWR018
 U 1 1 597403FE
 P 5750 7400
-F 0 "#PWR9" H 5750 7150 50  0001 C CNN
+F 0 "#PWR018" H 5750 7150 50  0001 C CNN
 F 1 "GND" H 5750 7250 50  0000 C CNN
 F 2 "" H 5750 7400 50  0001 C CNN
@@
 	9750 3400 9750 3900
 $Comp
-L GND #PWR17
+L GND #PWR019
 U 1 1 59753E6C
 P 9750 3900
-F 0 "#PWR17" H 9750 3650 50  0001 C CNN
+F 0 "#PWR019" H 9750 3650 50  0001 C CNN
 F 1 "GND" H 9750 3750 50  0000 C CNN
 F 2 "" H 9750 3900 50  0001 C CNN
@@
 F 0 "R4" V 730 1000 50  0000 C CNN
 F 1 "10KΩ" V 550 1000 50  0000 C CNN
-F 2 "Resistors_SMD:R_0805_HandSoldering" V 580 1000 50  0001 C CNN
+F 2 "Resistors_SMD:R_0805" V 580 1000 50  0001 C CNN
 F 3 "" H 650 1000 50  0001 C CNN
 	1    650  1000
@@
 Wire Wire Line
 	6400 3200 6300 3200
+$Comp
+L C_Small C7
+U 1 1 59933442
+P 2750 900
+F 0 "C7" H 2760 970 50  0000 L CNN
+F 1 "100nF" V 2650 950 50  0000 L CNN
+F 2 "Capacitors_SMD:C_0805" H 2750 900 50  0001 C CNN
+F 3 "" H 2750 900 50  0001 C CNN
+	1    2750 900
+	0    1    1    0
+$EndComp
+Wire Wire Line
+	2550 800  2550 950
+Wire Wire Line
+	2350 950  2350 800
+Wire Wire Line
+	2650 900  2550 900
+Connection ~ 2550 900
+$Comp
+L C_Small C6
+U 1 1 59933B83
+P 2150 900
+F 0 "C6" H 2160 970 50  0000 L CNN
+F 1 "100nF" V 2050 650 50  0000 L CNN
+F 2 "Capacitors_SMD:C_0805" H 2150 900 50  0001 C CNN
+F 3 "" H 2150 900 50  0001 C CNN
+	1    2150 900
+	0    1    1    0
+$EndComp
+Wire Wire Line
+	2250 900  2350 900
+Connection ~ 2350 900
+Wire Wire Line
+	2050 900  1900 900
+Wire Wire Line
+	2850 900  3000 900
+$Comp
+L GND #PWR020
+U 1 1 59933E8A
+P 3000 900
+F 0 "#PWR020" H 3000 650 50  0001 C CNN
+F 1 "GND" H 3000 750 50  0000 C CNN
+F 2 "" H 3000 900 50  0001 C CNN
+F 3 "" H 3000 900 50  0001 C CNN
+	1    3000 900
+	0    -1   -1   0
+$EndComp
+$Comp
+L GND #PWR021
+U 1 1 59933EF9
+P 1900 900
+F 0 "#PWR021" H 1900 650 50  0001 C CNN
+F 1 "GND" H 1900 750 50  0000 C CNN
+F 2 "" H 1900 900 50  0001 C CNN
+F 3 "" H 1900 900 50  0001 C CNN
+	1    1900 900
+	0    1    1    0
+$EndComp
 $EndSCHEMATC

Commit message: Enlarge some of the pads for hand soldering
Parts:
- C3, C4, C5: footprint Capacitors_SMD:C_0805 -> Capacitors_SMD:C_0805_HandSoldering
- R1, R2, R3, R6, R7: footprint Resistors_SMD:R_0805 -> Resistors_SMD:R_0805_HandSoldering
Changed lines of the file:
@@
 F 0 "C3" H 5625 1750 50  0000 L CNN
 F 1 "1uF" H 5625 1550 50  0000 L CNN
-F 2 "Capacitors_SMD:C_0805" H 5638 1500 50  0001 C CNN
+F 2 "Capacitors_SMD:C_0805_HandSoldering" H 5638 1500 50  0001 C CNN
 F 3 "" H 5600 1650 50  0001 C CNN
 F 4 "1276-6471-1-ND" H 5600 1650 60  0001 C CNN "Digikey"
@@
 F 0 "C4" H 7125 1750 50  0000 L CNN
 F 1 "1uF" H 7125 1550 50  0000 L CNN
-F 2 "Capacitors_SMD:C_0805" H 7138 1500 50  0001 C CNN
+F 2 "Capacitors_SMD:C_0805_HandSoldering" H 7138 1500 50  0001 C CNN
 F 3 "" H 7100 1650 50  0001 C CNN
 F 4 "Samsung Samsung CL21B105KOFNNNG" H 7100 1650 60  0001 C CNN "Part"
@@
 F 0 "R1" V 9150 1450 50  0000 L CNN
 F 1 "470Ω" V 9350 1500 50  0000 L CNN
-F 2 "Resistors_SMD:R_0805" H 9250 1500 50  0001 C CNN
+F 2 "Resistors_SMD:R_0805_HandSoldering" H 9250 1500 50  0001 C CNN
 F 3 "" H 9250 1500 50  0001 C CNN
 	1    9250 1500
@@
 F 0 "R2" V 9600 1450 50  0000 L CNN
 F 1 "470Ω" V 9800 1500 50  0000 L CNN
-F 2 "Resistors_SMD:R_0805" H 9700 1500 50  0001 C CNN
+F 2 "Resistors_SMD:R_0805_HandSoldering" H 9700 1500 50  0001 C CNN
 F 3 "" H 9700 1500 50  0001 C CNN
 	1    9700 1500
@@
 F 0 "R3" V 10050 1450 50  0000 L CNN
 F 1 "470Ω" V 10250 1500 50  0000 L CNN
-F 2 "Resistors_SMD:R_0805" H 10150 1500 50  0001 C CNN
+F 2 "Resistors_SMD:R_0805_HandSoldering" H 10150 1500 50  0001 C CNN
 F 3 "" H 10150 1500 50  0001 C CNN
 	1    10150 1500
@@
 F 0 "R6" V 5450 4900 50  0000 L CNN
 F 1 "10KΩ" V 5650 4850 50  0000 L CNN
-F 2 "Resistors_SMD:R_0805" H 5550 4950 50  0001 C CNN
+F 2 "Resistors_SMD:R_0805_HandSoldering" H 5550 4950 50  0001 C CNN
 F 3 "" H 5550 4950 50  0001 C CNN
 	1    5550 4950
@@
 F 0 "R7" V 5450 5250 50  0000 L CNN
 F 1 "10KΩ" V 5650 5200 50  0000 L CNN
-F 2 "Resistors_SMD:R_0805" H 5550 5300 50  0001 C CNN
+F 2 "Resistors_SMD:R_0805_HandSoldering" H 5550 5300 50  0001 C CNN
 F 3 "" H 5550 5300 50  0001 C CNN
 	1    5550 5300
@@
 F 0 "C5" H 5810 3920 50  0000 L CNN
 F 1 "100nF" H 5810 3770 50  0000 L CNN
-F 2 "Capacitors_SMD:C_0805" H 5800 3850 50  0001 C CNN
+F 2 "Capacitors_SMD:C_0805_HandSoldering" H 5800 3850 50  0001 C CNN
 F 3 "" H 5800 3850 50  0001 C CNN
 	1    5800 3850

Commit message: Add LDO Digikey part number
Parts:
- U4: Digikey (none) -> 296-40365-1-ND
Changed lines of the file:
@@
 F 2 "TO_SOT_Packages_SMD:SOT-23-6" H 6700 1750 50  0001 L CNN
 F 3 "" H 6300 1500 50  0001 C CNN
+F 4 "296-40365-1-ND" H 6300 1500 60  0001 C CNN "Digikey"
 	1    6300 1500
 	1    0    0    -1
